File: Capacitive Sensor.kicad_pcb (KiCad board)
At the start: 2 copper layers, 6 parts, among them J1 Conn_01x03, U1 TLC555

Commit message: update sensor
Parts:
- removed the REF** at (155.5, 106.8)
- added REF**: muwave_polygon, muwave_polygon, F.Cu at (160.5, 141.5)
- added REF**: muwave_polygon, muwave_polygon, F.Cu at (138.5, 143.5)
- moved C1 10.9 mm to (154.9, 94.5), turned to 90 degrees
- moved J1 8.50 mm to (150.0, 88.8)
- moved U1 7.52 mm to (150.1, 97.2), turned to 180 degrees
- moved R2 5.59 mm to (145.0, 96.0), turned to 90 degrees
- moved R1 2.77 mm to (145.0, 99.5), turned to 90 degrees
Routing:
- net C-: track 0.00 -> 33.1 mm, vias 0 -> 2
- net C+: track 0.00 -> 27.8 mm, vias 0 -> 2
- net 555_Output: track 0.00 -> 10.4 mm, vias 0 -> 2
- net Net-(R1-Pad2): track 0.00 -> 4.42 mm
- added copper zone on F.Cu, net +3V3
- added copper zone on B.Cu, net C-
Other:
- board outline added: 24.1 x 60.5 mm
- board text added: "->"
- board text added: "Designed By: Harry Dobbs"
